File: Kicad/isa_FDC-CF-USB.kicad_pcb (KiCad board)
At the start: 2 copper layers, 185.4 x 102.9 mm, 79 parts, among them J3 USB_A, P1 FLOPPY, P2 LED_USB, P3 CF_CARD, P4 LED_XTCF, SW1 XTCF_CFG, SW2 FDC_CFG, SW3 XTCF_ROM_CFG, U1 82077AA, U10 74LS04, U11 28C64, U12 74LS688, U13 74LS32, U14 74HC688, U15 74LS33, U16 CH375, U17 74HC688, U18 74HC245, U4 28C64, U5 74LS688, U6 74ALS138, U7 74ALS138, U9 74LS688, X1 24MHz, Y2 12MHz

Commit message: Add files via upload
Parts:
- removed the C11 at (225.4, 120.7)
- removed C30, C31: 22uF, My_Components:Cap_Tant_508
- removed C32: 0.01uF, My_Components:Cap_Cer_508
- removed C34: 100uF, My_Components:Cap_Tant_508
- removed C35, C36: 15pF, My_Components:Cap_Cer_508
- removed D2: LED_USB, My_Components:LED_3mm
- removed the JP2 at (56.5, 81.9)
- removed JP20, JP6: Jumper_2_Open, My_Components:Conn_Pin_Header_2x1_2.54mm_NoKey
- removed JP4: Jumper_2_Open, My_Components:Conn_Pin_Header_2x1_2.54mm
- removed JP5: USB_A0, My_Components:Conn_Pin_Header_2x1_2.54mm_NoKey
- removed the P2 at (55.2, 48.3)
- removed the R1 at (53.3, 54.6)
- removed R10: 2, My_Components:Res_762
- removed R120: 270, My_Components:Res_762
- removed R9: 10K, My_Components:Res_762
- removed the RR1 at (109.2, 48.9)
- removed the RR3 at (78.1, 48.9)
- removed the SW2 at (108.0, 42.5)
- removed U17: 74HC688, Package_DIP:DIP-20_W7.62mm
- added C19: 22pF, My_Components:Cap_Cer_508, F.Cu at (69.2, 56.7)
- added C20: 22pF, My_Components:Cap_Cer_508, F.Cu at (73.0, 56.7)
- added C21: 0.01uF, My_Components:Cap_Cer_508, F.Cu at (78.1, 56.5)
- added C23: 10uF, My_Components:Cap_Tant_508, F.Cu at (55.2, 79.4)
- added C24: 0.1uF, My_Components:Cap_Cer_508, F.Cu at (55.2, 71.8)
- added C25: 22pF, My_Components:Cap_Cer_508, F.Cu at (66.0, 44.5)
- added C26: 22pF, My_Components:Cap_Cer_508, F.Cu at (68.6, 44.5)
- added C27: 10uF, My_Components:Cap_Tant_508, F.Cu at (225.4, 117.5)
- added C28: 10uF, My_Components:Cap_Tant_508, F.Cu at (55.2, 123.2)
- added F1: 1.1A, My_Components:Cap_Cer_508, F.Cu at (55.2, 107.3)
- added FB1: FILTER, My_Components:Res_1016, F.Cu at (55.2, 89.5)
- added Q1: 2N7000, Package_TO_SOT_THT:TO-92, F.Cu at (86.4, 68.6)
- added R2: 330Ω, My_Components:Res_762, F.Cu at (55.2, 62.9)
- added RR2: 10kΩ, My_Components:Conn_SIL9, F.Cu at (108.0, 48.9)
- added RR4: 10kΩ, My_Components:Conn_SIL9, F.Cu at (108.0, 64.8)
- added SW1: FDC_CFG, My_Components:Switch_DIP_7_Positions, F.Cu at (109.2, 42.5)
- added SW4: USB_CFG, My_Components:Switch_DIP_4_Positions, F.Cu at (77.5, 42.5)
- added SW5: USB_IRQ, My_Components:Switch_DIP_5_Positions, F.Cu at (91.4, 42.5)
- added U13: 74ALS138, Package_DIP:DIP-16_W7.62mm, F.Cu at (67.9, 122.6)
- BUS1: value BUSPC_DEV -> PCB Edge Connector
- C11: renamed from C33; value 0.01uF -> 0.1uF
- C22: renamed from C37; value 100uF -> 10uF
- D1: value LED_XTCF -> PWR_LED
- JP3: value Jumper_2_Open -> LED_USB; footprint My_Components:Conn_Pin_Header_2x1_2.54mm_NoKey -> My_Components:Conn_Pin_Header_2x1_2.54mm
- P3: renamed from J3; footprint My_Components:Conn_Pin_Header_4x1_2.54mm -> My_Components:Conn_Pin_Header_5x1_2.54mm
- R6, R7: value 10K -> 1kΩ
- R8: value 10K -> 470Ω
- RR1: renamed from RR2; footprint Conn_SIL-6 -> My_Components:Conn_SIL6
- RR3: renamed from RR4; footprint Resistor_THT:R_Array_SIP4 -> My_Components:Conn_SIL5
- SW2: renamed from SW1; value XTCF_CFG -> XTCF_CS
- SW3: value XTCF_ROM_CFG -> XTCF_CFG
- U14: value 74HC688 -> 74LS32; footprint Package_DIP:DIP-20_W7.62mm -> Package_DIP:DIP-14_W7.62mm
- U15: value 74LS33 -> USBLC6-2P6; footprint Package_DIP:DIP-14_W7.62mm -> Package_TO_SOT_SMD:SOT-23-6
- moved U15 48.7 mm to (61.0, 43.2)
- moved C29 46.5 mm to (57.8, 48.3), turned to 90 degrees
- moved R8 38.8 mm to (55.2, 66.7), turned to 180 degrees
- moved P3 31.6 mm to (62.2, 38.7), turned to 0 degrees
- moved C22 27.9 mm to (55.2, 99.7), turned to 90 degrees
- moved SW2 27.8 mm to (94.0, 58.4)
- moved RR3 27.6 mm to (89.9, 64.8), turned to 180 degrees
- moved SW3 27.3 mm to (109.2, 58.4)
- moved JP3 26.7 mm to (55.2, 58.4), turned to 0 degrees
- moved C11 17.8 mm to (85.7, 76.2), turned to -90 degrees
- moved U10 15.9 mm to (101.6, 107.3)
- moved U7 15.9 mm to (113.0, 88.3)
- moved R7 13.2 mm to (83.2, 56.5), turned to 90 degrees
- moved JP2 10.2 mm to (55.2, 55.2)
- moved C15 7.76 mm to (228.0, 80.7), turned to 0 degrees
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- renumbered C8 to C1, C27 to C10, C26 to C12, C19 to C13, C28 to C14, C16 to C15, C15 to C16, C23 to C18, C4 to C2, C5 to C3, C6 to C4, C7 to C5, C22 to C6, C21 to C7, C18 to C8, C20 to C9, P4 to JP2, P3 to P2, R2 to R1, R4 to R3, R5 to R4, R3 to R5, U13 to U10, U16 to U11, U18 to U12, U4 to U2, U5 to U3, U6 to U4, U7 to U5, U11 to U6, U9 to U7, U12 to U8, U10 to U9, Y2 to X2
Connections:
- C22 pad 1: VCC -> Net-(C22-Pad1)
- D1 pad 1: Net-(D1-A) -> GND
- D1 pad 2: Net-(D1-K) -> Net-(D1-A)
- JP3 pad 1: Net-(JP3-A) -> Net-(JP3-P1)
- JP3 pad 2: Net-(JP3-B) -> /~{ACT}
- P3 pad 2: Net-(J3-D-) -> Net-(P3-D-)
- P3 pad 3: Net-(J3-D+) -> Net-(P3-D+)
- R6 pad 2: Net-(JP20-B) -> Net-(Q1-D)
- R7 pad 1: Net-(JP3-B) -> Net-(Q1-G)
- R7 pad 2: Net-(JP4-B) -> VCC
- R8 pad 2: Net-(R8-Pad2) -> Net-(JP3-P1)
- RR3 pad 2: Net-(U12-Q0) -> Net-(U8-Q2)
- RR3 pad 4: Net-(U12-Q2) -> Net-(U8-Q0)
- SW2 pad 1: Net-(U12-Q0) -> Net-(U8-Q0)
- SW2 pad 3: Net-(U12-Q2) -> Net-(U8-Q2)
- SW3 pad 2: /~{ROMW} -> /~{CF_ROMW}
- U10 pad 10: GND -> Net-(U10-Pad10)
- U10 pad 12: GND -> Net-(U10-Pad10)
- U10 pad 13: GND -> Net-(U10-Pad10)
- U10 pad 9: GND -> Net-(U10-Pad10)
- U11 pad 1: unconnected-(U16-~{INT}-Pad1) -> Net-(Q1-G)
- U11 pad 10: Net-(J3-D+) -> Net-(U11-UD+)
- U11 pad 11: Net-(J3-D-) -> Net-(U11-UD-)
- U11 pad 2: /RSTDRV -> /RESETDRV
- U11 pad 8: /A0-SEL -> /A0
- U14 pad 1: GND -> Net-(Q1-D)
- U14 pad 10: GND -> /AEN
- U14 pad 11: /A16 -> unconnected-(U14-Pad11)
- U14 pad 12: Net-(JP20-B) -> unconnected-(U14-Pad12)
- U14 pad 13: /A17 -> unconnected-(U14-Pad13)
- U14 pad 14: GND -> (no net)
- U14 pad 3: GND -> Net-(SW5-Pad10)
- U14 pad 4: GND -> Net-(SW4-Pad5)
- U14 pad 5: GND -> Net-(U14-Pad5)
- U14 pad 6: GND -> /~{USB-CS}
- U14 pad 7: GND -> (no net)
- U14 pad 8: /A15 -> Net-(U14-Pad5)
- U14 pad 9: VCC -> /A3
- U15 pad 1: Net-(R8-Pad2) -> Net-(U11-UD-)
- U15 pad 2: /~{SMEMR} -> GND
- U15 pad 3: Net-(JP3-B) -> Net-(U11-UD+)
- U15 pad 4: Net-(R9-Pad2) -> Net-(P3-D+)
- U15 pad 5: /~{IOR} -> VCC
- U15 pad 6: /~{USB-CS} -> Net-(P3-D-)
- U2 pad 1: /RDY/~{BUSY} -> /FDC_RDY/~{BUSY}
- U2 pad 20: /~{ROM_CS} -> /~{FDC_ROM_CS}
- U2 pad 27: /~{ROMW} -> /~{FDC_ROMW}
- U6 pad 1: /RDY/~{BUSY} -> /CF_RDY/~{BUSY}
- U6 pad 20: /~{ROM_CS} -> /~{CF_ROM_CS}
- U6 pad 27: /~{ROMW} -> /~{CF_ROMW}
- U7 pad 19: /~{ROM_CS} -> /~{CF_ROM_CS}
- U8 pad 3: Net-(U12-Q0) -> Net-(U8-Q0)
- U8 pad 7: Net-(U12-Q2) -> Net-(U8-Q2)
- U9 pad 10: Net-(D1-K) -> unconnected-(U9-Pad10)
- U9 pad 11: Net-(U10-Pad11) -> unconnected-(U9-Pad11)
- U9 pad 13: Net-(U10-Pad11) -> Net-(U9-Pad13)
- U9 pad 8: Net-(U10-Pad11) -> Net-(U9-Pad13)
Routing:
- net /~{ROM_CS}: track 185.7 -> 0.00 mm, vias 6 -> 0
- net /IRQ3: track 0.00 -> 157.3 mm, vias 0 -> 3
- net /~{ROMW}: track 149.8 -> 0.00 mm, vias 5 -> 0
- net /IRQ4: track 0.00 -> 149.5 mm, vias 0 -> 3
- net /IRQ5: track 0.00 -> 148.0 mm, vias 0 -> 3
- net /~{FDC_ROM_CS}: track 0.00 -> 145.6 mm, vias 0 -> 3
- net /IRQ7: track 0.00 -> 142.0 mm, vias 0 -> 5
- net /A1: track 322.3 -> 191.8 mm
- net /RDY/~{BUSY}: track 127.6 -> 0.00 mm, vias 4 -> 0
- net Net-(U12-Q2): track 115.9 -> 0.00 mm
- net /FDC_RDY/~{BUSY}: track 0.00 -> 114.2 mm, vias 0 -> 4
- net /~{FDC_ROMW}: track 0.00 -> 113.0 mm
- net Net-(U12-Q0): track 110.8 -> 0.00 mm
- net Net-(SW5-Pad10): track 0.00 -> 110.1 mm, vias 0 -> 1
- net /IRQ6: track 110.4 -> 217.2 mm
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Other:
- board text added: "FDC: Sergey Kiselev XT-CF lite 4.0c: Sergey Kiselev Merged and added CH375B USB-Storage: Peter Reichenbach"
- board text added: "SW1.1/SW3.1: ON: Enable ROM SW1.2/SW3.2: ON: Enable EEPROM write"
- board text added: "SW1.3/SW3.3 - SW1.7/SW3.7: ROM Address Selection 1 = ON; 0 = OFF"
- board text added: "SW1.8/SW3.8 - NOT USED"
- board text added: "SW2.1 - SW2.3: I/O Address Selection 1 = ON; 0 = OFF"
- board text added: "SW4.1 - ON: 230h SW4.2 - ON: 240h SW4.3 - ON: 250h SW4.4 - ON: 260h Only one switch can be ON at a time"
- board text added: "SW5.1 - ON: IRQ3 SW5.2 - ON: IRQ4 SW5.3 - ON: IRQ5 SW5.4 - ON: IRQ6 SW5.5 - ON: IRQ7 Only one switch can be ON at a time If everything OFF: no IRQ"
- board text removed: "01011 - 0xE8000 01010 - 0xEA000 01001 - 0xEC000 01000 - 0xEE000"
- board text removed: "DRIVE A: / B:"
- board text removed: "DRIVE C:"
- board text removed: "DRIVE D:"
- board text removed: "SW1.1 - SW1.3: I/O Address Selection 1 = ON; 0 = OFF"
- board text removed: "SW1.1 - SW1.4: Serial Port IRQ Selection SW1.1: ON: IRQ3 (COM2, COM4) SW1.3: ON: IRQ5 SW1.2: ON: IRQ4 (COM1, COM3) SW1.4: ON: IRQ7 SW1.5 - SW1.8: Serial Port I/O Address Selection SW1.5: ON: 0x2E8 (COM4) SW1.7: ON: 0x2F8 (COM2) SW1.6: ON: 0x3E8 (COM3) SW1.8: ON: 0x3F8 (COM1)"
- board text removed: "SW1.4 - NOT USED"
- board text removed: "SW2.1: ON: Enable ROM SW2.2: ON: Enable EEPROM write"
- board text removed: "SW2.3 - SW2.7: ROM Address Selection 1 = ON; 0 = OFF"
- board text removed: "SW2.8 - NOT USED"
