File: Kicad/isa_FDC-CF-USB.kicad_sch (KiCad schematic)
At the start: 101 parts, among them J3 USB_A, P1 FLOPPY, P2 LED_USB, P3 CF_CARD, P4 LED_XTCF, SW1 XTCF_CFG, SW2 FDC_CFG, SW3 XTCF_ROM_CFG, U1 82077AA, U10 74LS04, U11 28C64, U12 74LS688, U13 74LS32, U14 74HC688, U15 74LS33, U16 CH375, U17 74HC688, U18 74HC245, U4 28C64, U5 74LS688, U6 74ALS138, U7 74ALS138, U9 74LS688, X1 24MHz, Y2 12MHz

Commit message: Add files via upload
Parts:
- removed C39: 0.1uF, my_components:Cap_Cer_508, symbol 8088-FE2010A-SBC-rescue:C
- removed SW1: XTCF_CFG, My_Components:Switch_DIP_3_Positions, symbol Switch:SW_DIP_x03
- added SW1: CFG, my_components:Switch_DIP_3_Positions, symbol 8088-FE2010A-SBC-rescue:Switch_DIP_3_Positions
- SW3: value XTCF_ROM_CFG -> XTCF_CFG
Connections:
- net GND: now also SW1.4, SW1.5, SW1.6
- net at RR4.2, U12.3 (Q0): now also SW1.1
- net at RR4.3, U12.5 (Q1): now also SW1.2
- net at RR4.4, U12.7 (Q2): now also SW1.3
Other:
- note added: "CF INTERFACE"
- note added: "FDC BIOS ROM"
- note added: "FDC CHIP SELECT"
- note added: "FLOPPY DISK CONTROLLER"
- note added: "SW1.1 - ON: CF A7 = 0; OFF: CF A7 = 1 SW1.2 - ON: CF A6 = 0; OFF: CF A6 = 1 SW1.3 - ON: CF A5 = 0; OFF: CF A5 = 1"
- note added: "SW3.1 - ON: Enable ROM SW3.2 - ON: Enable EEPROM write SW3.3 - ON: ROM A17 = 0; OFF: ROM A17 = 1 SW3.4 - ON: ROM A16 = 0; OFF: ROM A16 = 1 SW3.5 - ON: ROM A15 = 0; OFF: ROM A15 = 1 SW3.6 - ON: ROM A14 = 0; OFF: ROM A14 = 1 SW3.7 - ON: ROM A13 = 0; OFF: ROM A13 = 1 SW3.8 - NOT USED"
- note added: "XT-CF BIOS ROM"
- note added: "XT-CF CHIP SELECT"
- note added: "XT-USB"
- note removed: "BIOS Extension ROM"
- note removed: "Compact Flash Interface"
- note removed: "Floppy Disk Controller"
- note removed: "I/O Ports Chip Select Logic"
- note removed: "SW1.1 - ON: CF A7 = 0; OFF: CF A7 = 1 SW1.2 - ON: CF A6 = 0; OFF: CF A6 = 1 SW1.3 - ON: CF A5 = 0; OFF: CF A5 = 1 SW1.4 - NOT USED SW2.1 - ON: Enable ROM SW2.2 - ON: Enable EEPROM write SW2.3 - ON: ROM A17 = 0; OFF: ROM A17 = 1 SW2.4 - ON: ROM A16 = 0; OFF: ROM A16 = 1 SW2.5 - ON: ROM A15 = 0; OFF: ROM A15 = 1 SW2.6 - ON: ROM A14 = 0; OFF: ROM A14 = 1 SW2.7 - ON: ROM A13 = 0; OFF: ROM A13 = 1 SW2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"
- note removed: "Settings"
- moved on the sheet: BUS1, C1, C10, C11, C12, C13, C14, C15, C16, C17, C18, C19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

Commit message: Add files via upload
Parts:
- removed C1, C10, C2, C3, C4, C5, C6, C7, C9: 0.1uF, symbol isa_fdc-rescue:C
- removed C11, C12, C13, C14: 10uF, symbol isa_fdc-rescue:CP1
- removed C15, C16: 22pF, symbol isa_fdc-rescue:C
- removed C17: 4.7nF, symbol isa_fdc-rescue:C
- removed C18, C19, C20, C21, C22, C23: 0.1uF, My_Components:Cap_Cer_508, symbol xt-cf-rescue:C
- removed C24, C25: 10uF, symbol xt-cf-rescue:CP1
- removed C26, C27, C28, C29: 0.1uF, My_Components:Cap_Cer_508, symbol Device:C
- removed C30, C31: 22uF, My_Components:Cap_Tant_508, symbol Device:CP1
- removed C32, C33: 0.01uF, My_Components:Cap_Cer_508, symbol Device:C
- removed C34: 100uF, My_Components:Cap_Tant_508, symbol Device:CP1
- removed C35, C36: 15pF, My_Components:Cap_Cer_508, symbol Device:C
- removed C8: 0.1uF, My_Components:Cap_Cer_508, symbol isa_fdc-rescue:C
- removed D2: LED_USB, My_Components:LED_3mm, symbol Device:LED
- removed JP2: USB_A1, My_Components:Conn_Pin_Header_2x1_2.54mm_NoKey, symbol Jumper:Jumper_2_Open
- removed JP20, JP3, JP6: Jumper_2_Open, My_Components:Conn_Pin_Header_2x1_2.54mm_NoKey, symbol Jumper:Jumper_2_Open
- removed JP4: Jumper_2_Open, My_Components:Conn_Pin_Header_2x1_2.54mm, symbol Jumper:Jumper_2_Open
- removed JP5: USB_A0, My_Components:Conn_Pin_Header_2x1_2.54mm_NoKey, symbol Jumper:Jumper_2_Open
- removed P2: LED_USB, My_Components:Conn_Pin_Header_2x1_2.54mm, symbol xt-cf-rescue:CONN_2
- removed R1: 330, My_Components:Res_762, symbol xt-cf-rescue:R
- removed R10: 2, My_Components:Res_762, symbol Device:R
- removed R120: 270, My_Components:Res_762, symbol Device:R
- removed R2: 470, My_Components:Res_762, symbol xt-cf-rescue:R
- removed R3: 1k, My_Components:Res_762, symbol xt-cf-rescue:R
- removed R4: 5.6k, My_Components:Res_762, symbol xt-cf-rescue:R
- removed R5: 10k, My_Components:Res_762, symbol xt-cf-rescue:R
- removed R6, R7, R8, R9: 10K, My_Components:Res_762, symbol Device:R
- removed RR1: 10k, My_Components:Conn_SIL9, symbol isa_fdc-rescue:RR9
- removed RR3: 10k, Resistor_THT:R_Array_SIP8, symbol xt-cf-rescue:RR9
- removed U14, U17: 74HC688, Package_DIP:DIP-20_W7.62mm, symbol 74xx:74HC688
- removed U15: 74LS33, Package_DIP:DIP-14_W7.62mm, symbol 74xx:74LS33
- removed Y2: 12MHz, My_Components:Crystal_HC-49U_Vert, symbol Device:Crystal
- added C1, C10, C11, C13, C9: 0.1uF, my_components:Cap_Cer_508, symbol 8088-FE2010A-SBC-rescue:C
- added C15, C16, C19, C20, C25, C26: 22pF, My_Components:Cap_Cer_508, symbol 8088-FE2010A-SBC-rescue:C
- added C21: 0.01uF, My_Components:Cap_Cer_508, symbol 8088-FE2010A-SBC-rescue:C
- added C23: 10uF, My_Components:Cap_Tant_508, symbol Device:CP1
- added C24, C29: 0.1uF, My_Components:Cap_Cer_508, symbol 8088-FE2010A-SBC-rescue:C
- added C27, C28: 10uF, My_Components:Cap_Tant_508, symbol 8088-FE2010A-SBC-rescue:C
- added F1: 1.1A, My_Components:Cap_Cer_508, symbol 8088-FE2010A-SBC-rescue:F_Small
- added FB1: FILTER, My_Components:Res_1016, symbol isa_svga-rescue:FILTER
- added JP3: LED_USB, My_Components:Conn_Pin_Header_2x1_2.54mm, symbol xt-cf-rescue:CONN_2
- added Q1: 2N7000, Package_TO_SOT_THT:TO-92, symbol Transistor_FET:BSS138
- added R1: 470Ω, my_components:Res_762, symbol 8088-FE2010A-SBC-rescue:R
- added R2: 330Ω, My_Components:Res_762, symbol 8088-FE2010A-SBC-rescue:R
- added R3: 5.6kΩ, my_components:Res_762, symbol 8088-FE2010A-SBC-rescue:R
- added R4: 10kΩ, my_components:Res_762, symbol 8088-FE2010A-SBC-rescue:R
- added R5: 1kΩ, my_components:Res_762, symbol 8088-FE2010A-SBC-rescue:R
- added R6, R7: 1kΩ, My_Components:Res_762, symbol 8088-FE2010A-SBC-rescue:R
- added R8: 470Ω, My_Components:Res_762, symbol 8088-FE2010A-SBC-rescue:R
- added RR2, RR4: 10kΩ, My_Components:Conn_SIL9, symbol 8088-FE2010A-SBC-rescue:RR9
- added SW4: USB_CFG, My_Components:Switch_DIP_4_Positions, symbol 8088-FE2010A-SBC-rescue:Switch_DIP_3_Positions
- added SW5: USB_IRQ, My_Components:Switch_DIP_5_Positions, symbol 8088-FE2010A-SBC-rescue:Switch_DIP_3_Positions
- added U13: 74ALS138, Package_DIP:DIP-16_W7.62mm, symbol isa_fdc-rescue:74LS138
- added U14: 74LS32, Package_DIP:DIP-14_W7.62mm, symbol 74xx:74LS32
- added U15: USBLC6-2P6, Package_TO_SOT_SMD:SOT-23-6, symbol Power_Protection:USBLC6-2P6
- added X2: 12MHz, symbol isa_fdc-rescue:CRYSTAL
- C17: value 0.1uF -> 4.7nF; footprint my_components:Cap_Cer_508 -> My_Components:Cap_Cer_508
- C22: renamed from C37; value 100uF -> 10uF
- D1: value LED_XTCF -> PWR_LED
- P3: renamed from J3; footprint My_Components:Conn_Pin_Header_4x1_2.54mm -> My_Components:Conn_Pin_Header_5x1_2.54mm
- RR1: renamed from RR2; footprint (none) -> My_Components:Conn_SIL6
- RR3: renamed from RR4; footprint Resistor_THT:R_Array_SIP4 -> My_Components:Conn_SIL5
- SW2: renamed from SW1; value CFG -> XTCF_CS
- renumbered C18 to C12, C40 to C18, C4 to C2, C5 to C3, C6 to C4, C7 to C5, C11 to C6, C9 to C7, C12 to C8, P4 to JP2, P3 to P2, SW2 to SW1, U13 to U10, U16 to U11, U18 to U12, U4 to U2, U5 to U3, U6 to U4, U7 to U5, U11 to U6, U9 to U7, U12 to U8, U10 to U9
Connections:
- net A0-SEL is gone; now on net A0: U11.8 (A0)
- net RSTDRV is gone; now on net RESETDRV: U11.2 (RESET)
- net A3: now also U14.9
- net A4: now also U13.1 (A)
- net A5: now also U13.2 (B)
- net A6: now also U13.3 (C)
- net A7: now also U13.5 (~{G2B})
- net A8: now also U13.4 (~{G2A})
- net A9: now also U13.6 (G1)
- net AEN: now also U14.10
- net CF_DMARQ: now also R3.2
- net CF_IORDY: now also R5.2
- net D7: now also R4.2
- net GND: now also D1.1 (K), C1.2, C10.2, C11.2, C13.2, C15.2, C16.2, C19.2, C20.2, C21.2, C23.2, C24.2, C25.2, C26.2, C27.2, C28.2, C29.2, C9.2, Q1.2 (S), R3.1, R4.1, U13.8 (GND), U14.2, U15.2 (GND); no longer C17.2, U10.10, U10.12, U10.13, U10.9
- net IRQ3: now also SW5.1
- net IRQ4: now also SW5.2
- net IRQ5: now also SW5.3
- net IRQ6: now also SW5.4
- net IRQ7: now also SW5.5
- net VCC: now also P2.38 (VCC), C1.1, C10.1, C11.1, C13.1, C27.1, C28.1, C29.1, C9.1, F1.2, R1.1, R2.1, R5.1, R6.1, R7.2, R8.1, RR2.1 (COM), RR4.1 (COM), U13.16 (VCC), U15.5 (VBUS); no longer C17.1, C22.1
- net ~{ACT}: now also JP3.2 (PM)
- net ~{USB-CS}: now also U14.6
- net at U1.33 (X1), X1.1: now also C16.1
- net at U1.34 (X2), X1.2: now also C15.1
- net at U1.37 (LOFIL): now also C17.2
- net at U1.38 (HIFIL): now also C17.1
- net at SW1.5, U3.12 (Q4): now also RR2.6
- net at SW1.6, U3.14 (Q5): now also RR2.7
- net at SW1.7, U3.16 (Q6): now also RR2.8
- net at SW1.3, U3.7 (Q2): now also RR2.4
- net at SW1.4, U3.9 (Q3): now also RR2.5
- net at D1.2 (A): now also R1.2; no longer U9.10
- net at JP2.1 (P1): now also R2.2
- net at SW3.1, U7.1 (~{G}): now also RR4.2
- net at SW3.3, U7.7 (Q2): now also RR4.4
- net at SW3.4, U7.9 (Q3): now also RR4.5
- net at SW3.5, U7.12 (Q4): now also RR4.6
- net at SW3.6, U7.14 (Q5): now also RR4.7
- net at SW3.7, U7.16 (Q6): now also RR4.8
- net at SW2.1, U8.3 (Q0): now also RR3.4; no longer RR3.2
- net at SW2.3, U8.7 (Q2): now also RR3.2; no longer RR3.4
- net at P3.1 (VBUS): now also C23.1, C24.1, FB1.1
- net at U11.13 (X1): now also C20.1, X2.2
- net at U11.14 (X0): now also C19.1, X2.1
- net at U9.13, U9.8: no longer U9.11
- net at U11.9 (U3): now also C21.1
- net at U11.1 (~{INT}): now also Q1.1 (G), R7.1
- net at U11.10 (UD+): now also C26.1, U15.3 (I/O2); no longer P3.3 (D+)
- net at U11.11 (UD-): now also C25.1, U15.1 (I/O1); no longer P3.2 (D-)
- net RDY/~{BUSY} renamed CF_RDY/~{BUSY}
- net CF_RDY/~{BUSY}: now also RR4.9; no longer U2.1 (RDY/~{BUSY})
- net ~{ROMW} renamed ~{CF_ROMW}
- net ~{CF_ROMW}: now also RR4.3; no longer SW1.2, U2.27 (~{WE})
- net ~{ROM_CS} renamed ~{CF_ROM_CS}
- net ~{CF_ROM_CS}: no longer SW1.1, U2.20 (~{CE})
- new net: U10.10, U10.12, U10.13, U10.9
- new net: SW4.1, U13.12 (~{Y3})
- new net: SW4.2, U13.11 (~{Y4})
- new net: SW4.3, U13.10 (~{Y5})
- new net: SW4.4, U13.9 (~{Y6})
- new net: SW4.5, SW4.6, SW4.7, SW4.8, U14.4
- new net: Q1.3 (D), R6.2, U14.1
- new net: JP3.1 (P1), R8.2
- new net: U14.5, U14.8
- new net: SW5.10, SW5.6, SW5.7, SW5.8, SW5.9, U14.3
- new net: P3.3 (D+), U15.4 (I/O2)
- new net: P3.2 (D-), U15.6 (I/O1)
- new net: C22.1, F1.1, FB1.2
- new net FDC_RDY/~{BUSY}: RR2.9, U2.1 (RDY/~{BUSY})
- new net ~{FDC_ROMW}: RR2.3, SW1.2, U2.27 (~{WE})
- new net ~{FDC_ROM_CS}: RR2.2, SW1.1, U2.20 (~{CE})
- no-connect marks 66 -> 67
Other:
- note added: "SW1.1 - ON: Enable ROM SW1.2 - ON: Enable EEPROM write SW1.3 - ON: ROM A17 = 0; OFF: ROM A17 = 1 SW1.4 - ON: ROM A16 = 0; OFF: ROM A16 = 1 SW1.5 - ON: ROM A15 = 0; OFF: ROM A15 = 1 SW1.6 - ON: ROM A14 = 0; OFF: ROM A14 = 1 SW1.7 - ON: ROM A13 = 0; OFF: ROM A13 = 1 SW1.8 - NOT USED"
- note added: "SW2.1 - ON: CF A7 = 0; OFF: CF A7 = 1 SW2.2 - ON: CF A6 = 0; OFF: CF A6 = 1 SW2.3 - ON: CF A5 = 0; OFF: CF A5 = 1"
- note added: "SW4.1 - ON: 230h SW4.2 - ON: 240h SW4.3 - ON: 250h SW4.4 - ON: 260h Only one switch can be ON at a time"
- note added: "SW5.1 - ON: IRQ3 SW5.2 - ON: IRQ4 SW5.3 - ON: IRQ5 SW5.4 - ON: IRQ6 SW5.5 - ON: IRQ7 Only one switch can be ON at a time If everything OFF: no IRQ"
- note removed: "Bypass Capacitors"
- note removed: "SW1.1 - ON: CF A7 = 0; OFF: CF A7 = 1 SW1.2 - ON: CF A6 = 0; OFF: CF A6 = 1 SW1.3 - ON: CF A5 = 0; OFF: CF A5 = 1"
- note removed: "SW2.1 - ON: Enable ROM SW2.2 - ON: Enable EEPROM write SW2.3 - ON: ROM A17 = 0; OFF: ROM A17 = 1 SW2.4 - ON: ROM A16 = 0; OFF: ROM A16 = 1 SW2.5 - ON: ROM A15 = 0; OFF: ROM A15 = 1 SW2.6 - ON: ROM A14 = 0; OFF: ROM A14 = 1 SW2.7 - ON: ROM A13 = 0; OFF: ROM A13 = 1 SW2.8 - NOT USED"
- title: ISA_FDC-CD-USB Card                                   V1.0 -> ISA_FDC-CF-USB Card                                   V1.0
- moved on the sheet: C12, C22, D1, P3, U11, U12, U9E, X1
